Commit message: Update handling of URDF / SRDF files

File: agimus_demo_05_pick_and_place/urdf/demo.urdf.xacro (robot description, xacro)
@@ -1,6 +1,6 @@
 <?xml version='1.0' encoding='utf-8'?>
 <robot xmlns:xacro="http://www.ros.org/wiki/xacro" name="panda">
-  <xacro:include filename="/home/gepetto/ros2_ws/src/agimus-demos/agimus_demo_05_pick_and_place/agimus_demo_05_pick_and_place/urdf/franka_robot.xacro"/>
-  <xacro:include filename="/home/gepetto/ros2_ws/src/agimus-demos/agimus_demo_05_pick_and_place/agimus_demo_05_pick_and_place/urdf/support.urdf.xacro"/>
+  <xacro:include filename="$(find agimus_demo_05_pick_and_place)/urdf/franka_robot.xacro"/>
+  <xacro:include filename="$(find agimus_demo_05_pick_and_place)/urdf/support.urdf.xacro"/>
   <xacro:support/>
   <xacro:franka_robot arm_id="panda"

File: agimus_demo_05_pick_and_place/urdf/franka_arm.xacro (robot description, xacro)
@@ -1,5 +1,5 @@
 <?xml version='1.0' encoding='utf-8'?>
 <robot xmlns:xacro="http://www.ros.org/wiki/xacro" name="panda">
-  <xacro:include filename="/home/gepetto/ros2_ws/src/agimus-demos/agimus_demo_05_pick_and_place/agimus_demo_05_pick_and_place/urdf/utils.xacro" />
+  <xacro:include filename="$(find agimus_demo_05_pick_and_place)/urdf/utils.xacro" />
   <!-- safety_distance: Minimum safety distance in [m] by which the collision volumes are expanded and which is enforced during robot motions -->
   <!-- arm_id: Namespace of the robot arm. Serves to differentiate between arms in case of multiple instances. -->

File: agimus_demo_05_pick_and_place/urdf/franka_robot.xacro (robot description, xacro)
@@ -9,7 +9,7 @@
     <!-- Is the robot being simulated in gazebo?" -->
     <xacro:arg name="gazebo" default="false" />
-    <xacro:include filename="/home/gepetto/ros2_ws/src/agimus-demos/agimus_demo_05_pick_and_place/agimus_demo_05_pick_and_place/urdf/utils.xacro" />
-    <xacro:include filename="/home/gepetto/ros2_ws/src/agimus-demos/agimus_demo_05_pick_and_place/agimus_demo_05_pick_and_place/urdf/franka_arm.xacro" />
-    <xacro:include filename="/home/gepetto/ros2_ws/src/agimus-demos/agimus_demo_05_pick_and_place/agimus_demo_05_pick_and_place/urdf/franka_hand.xacro"/>
+    <xacro:include filename="$(find agimus_demo_05_pick_and_place)/urdf/utils.xacro" />
+    <xacro:include filename="$(find agimus_demo_05_pick_and_place)/urdf/franka_arm.xacro" />
+    <xacro:include filename="$(find agimus_demo_05_pick_and_place)/urdf/franka_hand.xacro"/>
     <xacro:franka_arm arm_id="${arm_id}" safety_distance="0.03" gazebo="$(arg gazebo)" joint_limits="${joint_limits}"/>
     <xacro:franka_hand
@@ -24,5 +24,5 @@
     <!-- D435 camera -->
     <xacro:property name="camera_pose_file"
-                    value="/home/gepetto/ros2_ws/src/agimus-demos/agimus_demo_05_pick_and_place/agimus_demo_05_pick_and_place/calibrated-params.yaml" />
+                    value="$(find agimus_demo_05_pick_and_place)/config/calibrated-params.yaml" />
     <xacro:property name="camera_pose" value="${load_yaml(camera_pose_file)}"/>
     <link name="${arm_id}_ref_camera_link"/>
@@ -51,5 +51,5 @@
         <origin xyz="0.022 0 -0.012" rpy="3.141592653589793 0 -1.5707963267948966"/>
         <geometry>
-          <mesh filename="package://urdf/camera-support.stl" scale="1 1 1"/>
+          <mesh filename="package://agimus_demo_05_pick_and_place/urdf/meshes/camera-support.stl" scale="1 1 1"/>
         </geometry>
       </visual>
@@ -57,5 +57,5 @@
         <origin xyz="0.022 0 -0.012" rpy="3.141592653589793 0 -1.5707963267948966"/>
         <geometry>
-          <mesh filename="package://urdf/camera-support.stl" scale="1 1 1"/>
+          <mesh filename="package://agimus_demo_05_pick_and_place/urdf/meshes/camera-support.stl" scale="1 1 1"/>
         </geometry>
       </collision>

File: agimus_demo_05_pick_and_place/urdf/obj_01.urdf (robot description, URDF)
Before this commit: robot part, 1 links, 0 joints
Links:
- link base_link: geometry collision mesh filename=package://agimus_demo_05_pick_and_place/urdf/meshes/obj_01.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 scale=0.001 0.001 0.001; visual mesh filename=package://agimus_demo_05_pick_and_place/urdf/meshes/obj_01.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 scale=0.001 0.001 0.001

File: agimus_demo_05_pick_and_place/urdf/obj_23.urdf (robot description, URDF)
Before this commit: robot part, 1 links, 0 joints
Links:
- link base_link: geometry collision mesh filename=package://agimus_demo_05_pick_and_place/urdf/meshes/obj_23.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 scale=0.001 0.001 0.001; visual mesh filename=package://agimus_demo_05_pick_and_place/urdf/meshes/obj_23.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 scale=0.001 0.001 0.001
