Commit message: Fix some URDF and mesh paths.

File: agimus_demo_05_pick_and_place/urdf/franka_hand.xacro (robot description, xacro)
@@ -24,5 +24,5 @@
       <visual>
         <geometry>
-          <mesh filename="package://${description_pkg}/meshes/visual/finger.dae" />
+          <mesh filename="package://${description_pkg}/meshes/robot_ee/franka_hand_white/visual/finger.dae" />
         </geometry>
       </visual>
@@ -63,5 +63,5 @@
         <origin xyz="0 0 0" rpy="0 0 ${pi}" />
         <geometry>
-          <mesh filename="package://${description_pkg}/meshes/visual/finger.dae" />
+          <mesh filename="package://${description_pkg}/meshes/robot_ee/franka_hand_white/visual/finger.dae" />
         </geometry>
       </visual>

File: agimus_demo_05_pick_and_place/urdf/utils.xacro (robot description, xacro)
@@ -38,5 +38,5 @@
       <visual>
         <geometry>
-          <mesh filename="package://${description_pkg}/meshes/visual/${name}.dae" />
+          <mesh filename="package://${description_pkg}/meshes/robot_arms/fer/visual/${name}.dae" />
         </geometry>
       </visual>
