Commit message: initial commit on this branch

File: agimus_demo_05_pick_and_place/agimus_demo_05_pick_and_place/urdf/demo.urdf.xacro (robot description, xacro)
@@ -1,10 +1,33 @@
 <?xml version='1.0' encoding='utf-8'?>
-<robot xmlns:xacro="http://www.ros.org/wiki/xacro" name="panda">
-  <xacro:include filename="/home/gepetto/ros2_ws/src/agimus-demos/agimus_demo_05_pick_and_place/agimus_demo_05_pick_and_place/urdf/franka_robot.xacro"/>
-  <xacro:include filename="/home/gepetto/ros2_ws/src/agimus-demos/agimus_demo_05_pick_and_place/agimus_demo_05_pick_and_place/urdf/support.urdf.xacro"/>
-  <xacro:support/>
-  <xacro:franka_robot arm_id="panda"
+<robot xmlns:xacro="http://www.ros.org/wiki/xacro" name="fer">
+  <xacro:include filename="$(find franka_description)/robots/fer/fer.urdf.xacro">
+    <xacro:arg name="with_sc" value="true"/>  </xacro:include>
+  <!-- <xacro:support/>
+  <xacro:franka_robot arm_id="fer"
                       joint_limits="${xacro.load_yaml('$(find franka_description)/robots/fer/joint_limits.yaml')}">
-  </xacro:franka_robot>
-  <!-- wall behind the table -->
+  </xacro:franka_robot> -->
+  <link name="support_link">
+    <inertial>
+      <mass value="200"/>
+      <origin xyz="0 0 0"/>
+      <inertia ixx="50"  ixy="0"  ixz="0" iyy="50" iyz="0" izz="50" />
+    </inertial>
+    <visual>
+      <origin xyz="0 0 -1.0"/>
+      <geometry>
+        <box size="1.38 0.85 0.88"/>
+      </geometry>
+    </visual>
+    <collision>
+      <origin xyz="0 0 -1.0"/>
+      <geometry>
+        <box size="1.38 0.85 0.88"/>
+      </geometry>
+    </collision>
+  </link>
+  <joint name="support_joint" type="fixed">
+    <origin xyz="0.385 0 -1.44" rpy="0 0 0" />
+    <parent link="base" />
+    <child  link="support_link" />
+  </joint>
 </robot>

File: agimus_demo_05_pick_and_place/agimus_demo_05_pick_and_place/urdf/franka_hand.xacro (robot description, xacro)
@@ -24,5 +24,5 @@
       <visual>
         <geometry>
-          <mesh filename="package://${description_pkg}/meshes/visual/finger.dae" />
+          <mesh filename="package://${description_pkg}/meshes/robot_arms/fer/visual/finger.dae" />
         </geometry>
       </visual>
@@ -63,5 +63,5 @@
         <origin xyz="0 0 0" rpy="0 0 ${pi}" />
         <geometry>
-          <mesh filename="package://${description_pkg}/meshes/visual/finger.dae" />
+          <mesh filename="package://${description_pkg}/meshes/robot_arms/fer/visual/finger.dae" />
         </geometry>
       </visual>

File: agimus_demo_05_pick_and_place/agimus_demo_05_pick_and_place/urdf/franka_robot.xacro (robot description, xacro)
@@ -30,10 +30,11 @@
       <parent link="${arm_id}_hand"/>
       <child link="${arm_id}_ref_camera_link"/>
-      <origin xyz="${camera_pose['camera']['x']}
-                   ${camera_pose['camera']['y']}
-                   ${camera_pose['camera']['z']}"
-	      rpy="${camera_pose['camera']['roll']}
-                   ${camera_pose['camera']['pitch']}
-                   ${camera_pose['camera']['yaw']}"/>
+      <origin xyz="0.13967612678695326
+                  -0.014446642291159488
+                  -0.08527548627627562
+                "
+	      rpy="0.035422755166663634
+              -1.322907662418763
+              3.019794066851712"/>
     </joint>
     <xacro:include filename="$(find realsense2_description)/urdf/_d435.urdf.xacro" />
@@ -66,15 +67,4 @@
       <origin xyz="0 0 0" rpy="3.141592653589793 0 0"/>
     </joint>
-    <xacro:if value="$(arg gazebo)">
-      <xacro:include filename="$(find agimus_demos)/urdf/_d435.gazebo.xacro"/>
-      <xacro:gazebo_d435 camera_name="d435"
-                         reference_link="${arm_id}_ref_camera_link"
-                         topics_ns="camera"
-                         depth_optical_frame="camera_depth_optical_frame"
-                         color_optical_frame="camera_color_optical_frame"
-                         infrared1_optical_frame="camera_infrared1_optical_frame"
-                         infrared2_optical_frame="camera_infrared2_optical_frame">
-      </xacro:gazebo_d435>
-    </xacro:if>
     <!-- Define additional Gazebo tags -->
     <xacro:if value="$(arg gazebo)">

File: agimus_demo_05_pick_and_place/agimus_demo_05_pick_and_place/urdf/support.urdf.xacro (robot description, xacro)
@@ -1,187 +1,27 @@
 <?xml version='1.0' encoding='utf-8'?>
 <robot xmlns:xacro="http://www.ros.org/wiki/xacro">
-  <xacro:macro name="support" params="">
-      <link name="support_link">
-        <inertial>
-          <mass value="200"/>
-          <origin xyz="0 0 0.45"/>
-          <inertia ixx="50"  ixy="0"  ixz="0" iyy="50" iyz="0" izz="50" />
-        </inertial>
-        <visual>
-          <origin xyz="0 0 0.38"/>
-          <geometry>
-	    <box size="1.703 0.803 0.76"/>
-          </geometry>
-        </visual>
-        <collision>
-          <origin xyz="0 0 0.38"/>
-          <geometry>
-	    <box size="1.703 0.803 0.76"/>
-          </geometry>
-        </collision>
-        <!--visual>
-          <origin xyz="-0.61 0.2215 0.77"/>
-          <geometry>
-	    <box size="0.363 0.252 0.02"/>
-          </geometry>
-        </visual>
-        <collision>
-          <origin xyz="-0.61 0.2215 0.77"/>
-          <geometry>
-	    <box size="0.363 0.252 0.02"/>
-          </geometry>
-        </collision-->
-        <visual>
-          <origin xyz="0.6385 -0.1655 0.77"/>
-          <geometry>
-            <box size="0.3 0.3 0.02"/>
-          </geometry>
-        </visual>
-        <collision>
-          <origin xyz="0.6385 -0.1655 0.77"/>
-          <geometry>
-            <box size="0.3 0.3 0.02"/>
-          </geometry>
-        </collision>
-      </link>
-      <link name="wall_link_1">
-        <inertial>
-          <mass value="200"/>
-          <origin xyz="0 0 1."/>
-          <inertia ixx="50"  ixy="0"  ixz="0" iyy="50" iyz="0" izz="50" />
-        </inertial>
-        <visual>
-          <origin xyz="0 0 1.0"/>
-          <geometry>
-            <box size="3.0 0.1 2.0"/>
-          </geometry>
-        </visual>
-        <collision>
-          <origin xyz="0 0 1.0"/>
-          <geometry>
-            <box size="3.0 0.1 2.0"/>
-          </geometry>
-        </collision>
-      </link>
-      <link name="wall_link_2">
-        <inertial>
-          <mass value="200"/>
-          <origin xyz="0 0 1."/>
-          <inertia ixx="50"  ixy="0"  ixz="0" iyy="50" iyz="0" izz="50" />
-        </inertial>
-        <visual>
-          <origin xyz="0 0 1.0"/>
-          <geometry>
-            <box size="0.1 2.0 2.0"/>
-          </geometry>
-          <material name="lightGrey">
-            <color rgba="0.9 0.9 0.9 0.5"/>
-          </material>
-        </visual>
-        <collision>
-          <origin xyz="0 0 1.0"/>
-          <geometry>
-            <box size="0.1 2.0 2.0"/>
-          </geometry>
-        </collision>
-      </link>
-      <link name="wall_link_3">
-        <inertial>
-          <mass value="200"/>
-          <origin xyz="0 0 1."/>
-          <inertia ixx="50"  ixy="0"  ixz="0" iyy="50" iyz="0" izz="50" />
-        </inertial>
-        <visual>
-          <origin xyz="0 0 1.0"/>
-          <geometry>
-            <box size="0.7 0.12 2.0"/>
-          </geometry>
-        </visual>
-        <collision>
-          <origin xyz="0 0 1.0"/>
-          <geometry>
-            <box size="0.7 0.12 2.0"/>
-          </geometry>
-        </collision>
-      </link>
-      <link name="pedestal">
-        <inertial>
-          <mass value="1."/>
-          <origin xyz="1.05 0.45 0.4625"/>
-          <inertia ixx=".01" iyy=".01" izz=".1" ixy="0" ixz="0" iyz="0"/>
-        </inertial>
-        <visual>
-          <origin xyz="0 0 0.4625"/>
-          <geometry>
-            <box size="0.25 0.25 0.925"/>
-          </geometry>
-        </visual>
-        <collision>
-          <origin xyz="0 0 0.4625"/>
-          <geometry>
-            <box size="0.25 0.25 0.925"/>
-          </geometry>
-        </collision>
-      </link>
-      <!-- Wrap panda1 robot into a box shaped obstacle -->
-      <link name="panda1_box">
-        <inertial>
-          <mass value="100"/>
-          <origin xyz="0 0 0"/>
-          <inertia ixx="25"  ixy="0"  ixz="0" iyy="25" iyz="0" izz="25" />
-        </inertial>
-        <collision>
-          <origin xyz="0 0 0"/>
-          <geometry>
-            <box size="0.44 0.803 0.80"/>
-          </geometry>
-        </collision>
-        <visual>
-          <origin xyz="0 0 0"/>
-          <geometry>
-            <box size="0.44 0.803 0.80"/>
-          </geometry>
-          <material name="lightGrey">
-            <color rgba="0.9 0.9 0.9 0.5"/>
-          </material>
-        </visual>
-      </link>
-      <!-- Gazebo requires a joint to a link called "world" for statically mounted robots -->
-      <link name="world" />
-      <joint name="world_joint" type="fixed">
-        <origin xyz="0 0 0" rpy="0 0 0" />
-        <parent link="world" />
-        <child  link="support_link" />
-      </joint>
-      <joint name="support_joint" type="fixed">
-        <origin xyz="0.563 -0.1655 .78" rpy="0 0 ${pi}" />
-        <parent link="support_link" />
-        <child  link="panda_link0" />
-      </joint>
-      <joint name="wall_joint_1" type="fixed">
-        <origin xyz="0 1.07 0" />
-        <parent link="world"/>
-        <child link="wall_link_1"/>
-      </joint>
-      <joint name="wall_joint_2" type="fixed">
-        <origin xyz="1.78 0 0" />
-        <parent link="world"/>
-        <child link="wall_link_2"/>
-      </joint>
-      <joint name="wall_joint_3" type="fixed">
-        <origin xyz="1.40 0.96 0" />
-        <parent link="world"/>
-        <child link="wall_link_3"/>
-      </joint>
-      <joint name="pedestal_joint" type="fixed">
-        <origin xyz="1.05 0 0"/>
-        <parent link="world"/>
-        <child link="pedestal"/>
-      </joint>
-      <joint name="panda1_box_joint" type="fixed">
-        <origin xyz="-0.6315 0 1.17" />
-        <parent link="world"/>
-        <child link="panda1_box"/>
-      </joint>
-  </xacro:macro>
+  <link name="support_link">
+    <inertial>
+      <mass value="200"/>
+      <origin xyz="0 0 0"/>
+      <inertia ixx="50"  ixy="0"  ixz="0" iyy="50" iyz="0" izz="50" />
+    </inertial>
+    <visual>
+      <origin xyz="0 0 0"/>
+      <geometry>
+        <box size="1.38 0.85 0.88"/>
+      </geometry>
+    </visual>
+    <collision>
+      <origin xyz="0 0 0"/>
+      <geometry>
+        <box size="1.38 0.85 0.88"/>
+      </geometry>
+    </collision>
+  </link>
+  <joint name="support_joint" type="fixed">
+    <origin xyz="0.385 0 -1.44" rpy="0 0 0" />
+    <parent link="base" />
+    <child  link="support_link" />
+  </joint>
 </robot>

Commit message: small update to bring things to were they should be

File: agimus_demo_05_pick_and_place/agimus_demo_05_pick_and_place/urdf/demo.urdf.xacro (robot description, xacro)
@@ -14,5 +14,5 @@
     </inertial>
     <visual>
-      <origin xyz="0 0 -1.0"/>
+      <origin xyz="0 0 -0.44"/>
       <geometry>
         <box size="1.38 0.85 0.88"/>
@@ -20,5 +20,5 @@
     </visual>
     <collision>
-      <origin xyz="0 0 -1.0"/>
+      <origin xyz="0 0 -0.44"/>
       <geometry>
         <box size="1.38 0.85 0.88"/>

Commit message: Adding different verbose in hope to catch the problem

File: agimus_demo_05_pick_and_place/agimus_demo_05_pick_and_place/urdf/demo.urdf.xacro (robot description, xacro)
@@ -14,5 +14,5 @@
     </inertial>
     <visual>
-      <origin xyz="0 0 -0.44"/>
+      <origin xyz="0 0 0"/>
       <geometry>
         <box size="1.38 0.85 0.88"/>
@@ -20,5 +20,5 @@
     </visual>
     <collision>
-      <origin xyz="0 0 -0.44"/>
+      <origin xyz="0 0 0"/>
       <geometry>
         <box size="1.38 0.85 0.88"/>
@@ -27,5 +27,5 @@
   </link>
   <joint name="support_joint" type="fixed">
-    <origin xyz="0.385 0 -1.44" rpy="0 0 0" />
+    <origin xyz="0.385 0 -0.44" rpy="0 0 0" />
     <parent link="base" />
     <child  link="support_link" />

Commit message: Saving files for further experiment on this

File: agimus_demo_05_pick_and_place/agimus_demo_05_pick_and_place/urdf/demo.urdf.xacro (robot description, xacro)
@@ -1,33 +1,10 @@
 <?xml version='1.0' encoding='utf-8'?>
 <robot xmlns:xacro="http://www.ros.org/wiki/xacro" name="fer">
-  <xacro:include filename="$(find franka_description)/robots/fer/fer.urdf.xacro">
-    <xacro:arg name="with_sc" value="true"/>  </xacro:include>
-  <!-- <xacro:support/>
+  <xacro:include filename="/home/gepetto/ros2_ws/src/agimus-demos/agimus_demo_05_pick_and_place/agimus_demo_05_pick_and_place/urdf/franka_robot.xacro"/>
+  <xacro:include filename="/home/gepetto/ros2_ws/src/agimus-demos/agimus_demo_05_pick_and_place/agimus_demo_05_pick_and_place/urdf/support.urdf.xacro"/>
+  <xacro:support/>
   <xacro:franka_robot arm_id="fer"
                       joint_limits="${xacro.load_yaml('$(find franka_description)/robots/fer/joint_limits.yaml')}">
-  </xacro:franka_robot> -->
-  <link name="support_link">
-    <inertial>
-      <mass value="200"/>
-      <origin xyz="0 0 0"/>
-      <inertia ixx="50"  ixy="0"  ixz="0" iyy="50" iyz="0" izz="50" />
-    </inertial>
-    <visual>
-      <origin xyz="0 0 0"/>
-      <geometry>
-        <box size="1.38 0.85 0.88"/>
-      </geometry>
-    </visual>
-    <collision>
-      <origin xyz="0 0 0"/>
-      <geometry>
-        <box size="1.38 0.85 0.88"/>
-      </geometry>
-    </collision>
-  </link>
-  <joint name="support_joint" type="fixed">
-    <origin xyz="0.385 0 -0.44" rpy="0 0 0" />
-    <parent link="base" />
-    <child  link="support_link" />
-  </joint>
+  </xacro:franka_robot>
+  <!-- wall behind the table -->
 </robot>

File: agimus_demo_05_pick_and_place/agimus_demo_05_pick_and_place/urdf/franka_arm.xacro (robot description, xacro)
@@ -1,9 +1,9 @@
 <?xml version='1.0' encoding='utf-8'?>
-<robot xmlns:xacro="http://www.ros.org/wiki/xacro" name="panda">
+<robot xmlns:xacro="http://www.ros.org/wiki/xacro" name="fer">
   <xacro:include filename="/home/gepetto/ros2_ws/src/agimus-demos/agimus_demo_05_pick_and_place/agimus_demo_05_pick_and_place/urdf/utils.xacro" />
   <!-- safety_distance: Minimum safety distance in [m] by which the collision volumes are expanded and which is enforced during robot motions -->
   <!-- arm_id: Namespace of the robot arm. Serves to differentiate between arms in case of multiple instances. -->
   <!-- joint_limits: description of the joint limits that comes from a YAML file. Example definition: ${xacro.load_yaml('$(find franka_description)/robots/fr3/joint_limits.yaml')} -->
-  <xacro:macro name="franka_arm" params="arm_id:='panda' description_pkg:='franka_description' connected_to:='' xyz:='0 0 0' rpy:='0 0 0' gazebo:=false safety_distance:=0 joint_limits" >
+  <xacro:macro name="franka_arm" params="arm_id:='fer' description_pkg:='franka_description' connected_to:='' xyz:='0 0 0' rpy:='0 0 0' gazebo:=false safety_distance:=0 joint_limits" >
     <xacro:unless value="${not connected_to}">
       <joint name="${arm_id}_joint_${connected_to}" type="fixed">

File: agimus_demo_05_pick_and_place/agimus_demo_05_pick_and_place/urdf/support.urdf.xacro (robot description, xacro)
@@ -1,27 +1,187 @@
 <?xml version='1.0' encoding='utf-8'?>
 <robot xmlns:xacro="http://www.ros.org/wiki/xacro">
-  <link name="support_link">
-    <inertial>
-      <mass value="200"/>
-      <origin xyz="0 0 0"/>
-      <inertia ixx="50"  ixy="0"  ixz="0" iyy="50" iyz="0" izz="50" />
-    </inertial>
-    <visual>
-      <origin xyz="0 0 0"/>
-      <geometry>
-        <box size="1.38 0.85 0.88"/>
-      </geometry>
-    </visual>
-    <collision>
-      <origin xyz="0 0 0"/>
-      <geometry>
-        <box size="1.38 0.85 0.88"/>
-      </geometry>
-    </collision>
-  </link>
-  <joint name="support_joint" type="fixed">
-    <origin xyz="0.385 0 -1.44" rpy="0 0 0" />
-    <parent link="base" />
-    <child  link="support_link" />
-  </joint>
+  <xacro:macro name="support" params="">
+      <link name="support_link">
+        <inertial>
+          <mass value="200"/>
+          <origin xyz="0 0 0.45"/>
+          <inertia ixx="50"  ixy="0"  ixz="0" iyy="50" iyz="0" izz="50" />
+        </inertial>
+        <visual>
+          <origin xyz="0 0 0.38"/>
+          <geometry>
+	    <box size="1.703 0.803 0.76"/>
+          </geometry>
+        </visual>
+        <collision>
+          <origin xyz="0 0 0.38"/>
+          <geometry>
+	    <box size="1.703 0.803 0.76"/>
+          </geometry>
+        </collision>
+        <!--visual>
+          <origin xyz="-0.61 0.2215 0.77"/>
+          <geometry>
+	    <box size="0.363 0.252 0.02"/>
+          </geometry>
+        </visual>
+        <collision>
+          <origin xyz="-0.61 0.2215 0.77"/>
+          <geometry>
+	    <box size="0.363 0.252 0.02"/>
+          </geometry>
+        </collision-->
+        <visual>
+          <origin xyz="0.6385 -0.1655 0.77"/>
+          <geometry>
+            <box size="0.3 0.3 0.02"/>
+          </geometry>
+        </visual>
+        <collision>
+          <origin xyz="0.6385 -0.1655 0.77"/>
+          <geometry>
+            <box size="0.3 0.3 0.02"/>
+          </geometry>
+        </collision>
+      </link>
+      <link name="wall_link_1">
+        <inertial>
+          <mass value="200"/>
+          <origin xyz="0 0 1."/>
+          <inertia ixx="50"  ixy="0"  ixz="0" iyy="50" iyz="0" izz="50" />
+        </inertial>
+        <visual>
+          <origin xyz="0 0 1.0"/>
+          <geometry>
+            <box size="3.0 0.1 2.0"/>
+          </geometry>
+        </visual>
+        <collision>
+          <origin xyz="0 0 1.0"/>
+          <geometry>
+            <box size="3.0 0.1 2.0"/>
+          </geometry>
+        </collision>
+      </link>
+      <link name="wall_link_2">
+        <inertial>
+          <mass value="200"/>
+          <origin xyz="0 0 1."/>
+          <inertia ixx="50"  ixy="0"  ixz="0" iyy="50" iyz="0" izz="50" />
+        </inertial>
+        <visual>
+          <origin xyz="0 0 1.0"/>
+          <geometry>
+            <box size="0.1 2.0 2.0"/>
+          </geometry>
+          <material name="lightGrey">
+            <color rgba="0.9 0.9 0.9 0.5"/>
+          </material>
+        </visual>
+        <collision>
+          <origin xyz="0 0 1.0"/>
+          <geometry>
+            <box size="0.1 2.0 2.0"/>
+          </geometry>
+        </collision>
+      </link>
+      <link name="wall_link_3">
+        <inertial>
+          <mass value="200"/>
+          <origin xyz="0 0 1."/>
+          <inertia ixx="50"  ixy="0"  ixz="0" iyy="50" iyz="0" izz="50" />
+        </inertial>
+        <visual>
+          <origin xyz="0 0 1.0"/>
+          <geometry>
+            <box size="0.7 0.12 2.0"/>
+          </geometry>
+        </visual>
+        <collision>
+          <origin xyz="0 0 1.0"/>
+          <geometry>
+            <box size="0.7 0.12 2.0"/>
+          </geometry>
+        </collision>
+      </link>
+      <link name="pedestal">
+        <inertial>
+          <mass value="1."/>
+          <origin xyz="1.05 0.45 0.4625"/>
+          <inertia ixx=".01" iyy=".01" izz=".1" ixy="0" ixz="0" iyz="0"/>
+        </inertial>
+        <visual>
+          <origin xyz="0 0 0.4625"/>
+          <geometry>
+            <box size="0.25 0.25 0.925"/>
+          </geometry>
+        </visual>
+        <collision>
+          <origin xyz="0 0 0.4625"/>
+          <geometry>
+            <box size="0.25 0.25 0.925"/>
+          </geometry>
+        </collision>
+      </link>
+      <!-- Wrap fer1 robot into a box shaped obstacle -->
+      <link name="fer1_box">
+        <inertial>
+          <mass value="100"/>
+          <origin xyz="0 0 0"/>
+          <inertia ixx="25"  ixy="0"  ixz="0" iyy="25" iyz="0" izz="25" />
+        </inertial>
+        <collision>
+          <origin xyz="0 0 0"/>
+          <geometry>
+            <box size="0.44 0.803 0.80"/>
+          </geometry>
+        </collision>
+        <visual>
+          <origin xyz="0 0 0"/>
+          <geometry>
+            <box size="0.44 0.803 0.80"/>
+          </geometry>
+          <material name="lightGrey">
+            <color rgba="0.9 0.9 0.9 0.5"/>
+          </material>
+        </visual>
+      </link>
+      <!-- Gazebo requires a joint to a link called "world" for statically mounted robots -->
+      <link name="world" />
+      <joint name="world_joint" type="fixed">
+        <origin xyz="0 0 0" rpy="0 0 0" />
+        <parent link="world" />
+        <child  link="support_link" />
+      </joint>
+      <joint name="support_joint" type="fixed">
+        <origin xyz="0.563 -0.1655 .78" rpy="0 0 ${pi}" />
+        <parent link="support_link" />
+        <child  link="fer_link0" />
+      </joint>
+      <joint name="wall_joint_1" type="fixed">
+        <origin xyz="0 1.07 0" />
+        <parent link="world"/>
+        <child link="wall_link_1"/>
+      </joint>
+      <joint name="wall_joint_2" type="fixed">
+        <origin xyz="1.78 0 0" />
+        <parent link="world"/>
+        <child link="wall_link_2"/>
+      </joint>
+      <joint name="wall_joint_3" type="fixed">
+        <origin xyz="1.40 0.96 0" />
+        <parent link="world"/>
+        <child link="wall_link_3"/>
+      </joint>
+      <joint name="pedestal_joint" type="fixed">
+        <origin xyz="1.05 0 0"/>
+        <parent link="world"/>
+        <child link="pedestal"/>
+      </joint>
+      <joint name="fer1_box_joint" type="fixed">
+        <origin xyz="-0.6315 0 1.17" />
+        <parent link="world"/>
+        <child link="fer1_box"/>
+      </joint>
+  </xacro:macro>
 </robot>
