Commit message: Update support and foam block to match with Prague setup

File: agimus_demo_06_regrasp/urdf/support.urdf.xacro (robot description, xacro)
@@ -140,5 +140,5 @@
         <origin xyz="0 0 0.0225" />
         <geometry>
-          <box size="0.2 0.4 0.045" />
+          <box size="0.5 0.9 0.045" />
         </geometry>
         <material name="transp_blue">
@@ -149,5 +149,5 @@
         <origin xyz="0 0 0.0225" />
         <geometry>
-          <box size="0.2 0.4 0.045" />
+          <box size="0.5 0.9 0.045" />
         </geometry>
       </collision>
